Commit message: latest

File: ros_ws/src/my_bot/description/camera.xacro (robot description, xacro)
@@ -1,4 +1,5 @@
 <?xml version="1.0"?>
 <robot xmlns:xacro="http://www.ros.org/wiki/xacro" >
+    <!-- ================= FRONT CAMERA ================= -->
     <joint name="camera_joint" type="fixed">
         <parent link="chassis"/>
@@ -30,10 +31,10 @@
                 <image>
                     <format>R8G8B8</format>
-                    <width>640</width>
-                    <height>480</height>
+                    <width>800</width>
+                    <height>800</height>
                 </image>
                 <clip>
                     <near>0.05</near>
-                    <far>8.0</far>
+                    <far>20.0</far>
                 </clip>
             </camera>
@@ -43,3 +44,47 @@
         </sensor>
     </gazebo>
+    <!-- ================= TOP DOWN CAMERA ================= -->
+    <joint name="top_camera_joint" type="fixed">
+        <parent link="chassis"/>
+        <child link="top_camera_link"/>
+        <!-- 4 meters above robot, rotated downward -->
+        <origin xyz="0 0 10.0" rpy="0 1.5708 0"/>
+    </joint>
+    <link name="top_camera_link">
+        <visual>
+            <geometry>
+                <box size="0.010 0.03 0.03"/>
+            </geometry>
+            <material name="blue"/>
+        </visual>
+    </link>
+    <joint name="top_camera_optical_joint" type="fixed">
+        <parent link="top_camera_link"/>
+        <child link="top_camera_link_optical"/>
+        <origin xyz="0 0 0" rpy="${-pi/2} 0 ${-pi/2}"/>
+    </joint>
+    <link name="top_camera_link_optical"></link>
+    <gazebo reference="top_camera_link">
+        <material>Gazebo/Blue</material>
+        <sensor name="top_camera" type="camera">
+            <pose>0 0 0 0 0 0</pose>
+            <visualize>true</visualize>
+            <update_rate>15</update_rate>
+            <camera>
+                <horizontal_fov>1.3</horizontal_fov>
+                <image>
+                    <format>R8G8B8</format>
+                    <width>800</width>
+                    <height>800</height>
+                </image>
+                <clip>
+                    <near>0.1</near>
+                    <far>20.0</far>
+                </clip>
+            </camera>
+            <plugin name="top_camera_controller" filename="libgazebo_ros_camera.so">
+                <frame_name>top_camera_link_optical</frame_name>
+            </plugin>
+        </sensor>
+    </gazebo>
 </robot>

Commit message: overall

File: ros_ws/src/my_bot/description/camera.xacro (robot description, xacro)
@@ -48,6 +48,5 @@
         <parent link="chassis"/>
         <child link="top_camera_link"/>
-        <!-- 4 meters above robot, rotated downward -->
-        <origin xyz="0 0 10.0" rpy="0 1.5708 0"/>
+        <origin xyz="0 0 15.0" rpy="0 1.5708 0"/>
     </joint>
     <link name="top_camera_link">

File: ros_ws/src/my_bot/description/lidar.xacro (robot description, xacro)
@@ -1,5 +1,4 @@
 <?xml version="1.0"?>
 <robot xmlns:xacro="http://www.ros.org/wiki/xacro">
-    <!-- LIDAR JOINT-->
     <joint name="laser_joint" type="fixed">
         <parent link="chassis"/>
@@ -28,5 +27,4 @@
     <visualize>true</visualize>
     <update_rate>10</update_rate>
-    <!-- THIS IS CRITICAL -->
     <frame>laser_frame</frame>
     <ray>
@@ -47,7 +45,8 @@
     <plugin name="laser_controller" filename="libgazebo_ros_ray_sensor.so">
         <ros>
-        <namespace>/</namespace>
-        <remapping>~/out:=/scan</remapping>
+            <namespace>/</namespace>
+            <remapping>~/out:=/scan</remapping>
         </ros>
+        <output_type>sensor_msgs/LaserScan</output_type>
         <frame_name>laser_frame</frame_name>
     </plugin>
